File: 2nd to final draft.sch (EAGLE design)
At the start: 61 parts, among them Q1 NPN 40V 1A SOT-23, U1 WS2812

Commit message: sd card fully laid out
Parts:
- added ATMEGA328P-AU1: ATMEGA328P-AU, Atmega-328pu:ATMEGA328P-AU
- added C14, C17, C18, C21, C22: .1uF, SparkFun-Retired:.22UF-CER
- added C16: .01 uF, SparkFun-Retired:.22UF-CER
- added C19: 10nF, SparkFun-Retired:.22UF-CER
- added C20: 2.2nF, SparkFun-Retired:.22UF-CER
- added C23, C24: 47pF, SparkFun-Retired:.22UF-CER
- added C25, C26, C28: 10uF, SparkFun-Retired:10UF-TANT
- added C27: 47uF, SparkFun-Retired:10UF-TANT
- added D6: 700mA/40V/533mV, SparkFun-DiscreteSemi:DIODE-SCHOTTKY-ZLLS500
- added FTDI231XS2: FT231XS, SparkFun-IC-Comms:FT231XS
- added IC3, IC6: 74ABT125PW, 74xx-us:74ABT125PW
- added IC4, IC5: (no value), linear-technology:LT1129CST5
- added J1: (no value), SparkFun-Connectors:USB_MICRO-B_SMT
- added J7_5V_BACKUP1: (no value), SparkFun-Connectors:CONN_01
- added J7_TMP3: (no value), SparkFun-Connectors:CONN_02LOCK
- added JP2: JUMPER-SMT_2_NO_NO-SILK_ROUND, SparkFun-Jumpers:JUMPER-SMT_2_NO_NO-SILK_ROUND
- added MPU1: MPU-6050, KevinKuwata1:MPU-6050
- added R14, R16, R17, R18, R19, R20, R25: 10k, SparkFun-Resistors:0.05OHM-0603-1/5W-1%
- added R21, R22: 27, SparkFun-Resistors:0.05OHM-0603-1/5W-1%
- added R23, R24: 1k, SparkFun-Resistors:0.05OHM-0603-1/5W-1%
- added S2: TAC_SWITCHSMD, SparkFun-Retired:TAC_SWITCHSMD
- added U$3: 1N7002PW, KevinKuwata1:1N7002PW
- added U$4: WM6698TR-ND_MICROSD, KevinKuwata1:WM6698TR-ND_MICROSD
- added Y2: (no value), SparkFun-Clocks:RESONATORSMD-7.4X3.4
Connections:
- new net N$10: IC3B.O, U$2.DAT1
- new net N$11: IC3C.O, U$2.CMD
- new net N$32: ATMEGA328P-AU1.AREF, C16.1
- new net N$33: ATMEGA328P-AU1.PB6, Y2.1
- new net N$34: ATMEGA328P-AU1.PB7, Y2.3
- new net N$35: C20.1, MPU1.CPOUT
- new net N$36: C18.1, MPU1.REGOUT
- new net N$37: C19.1, MPU1.VLOG
- new net N$38: C23.1, J1.D+, R21.1
- new net N$39: C24.1, J1.D-, R22.1
- new net N$40: FTDI231XS2.USBDP, R22.2
- new net N$41: FTDI231XS2.USBDM, R21.2
- new net N$42: C25.+, FTDI231XS2.VCC
- new net N$43: D6.A, J7_TMP3.1
- new net N$44: C26.+, IC4G$1.OUT, J7_5V_BACKUP1.1, JP2.2
- new net N$45: U$4.G1, U$4.G4
- new net N$46: IC6A.O, U$4.CLK
- new net N$47: IC6B.O, U$4.DAT1
- new net N$48: IC6C.O, U$4.CMD
- new net N$8: U$2.G1, U$2.G4
- new net N$9: IC3A.O, U$2.CLK
- net 3.3V: now also ATMEGA328P-AU1.GND, ATMEGA328P-AU1.GND_2, ATMEGA328P-AU1.GND_3, C16.2, C17.2, C18.2, C19.2, C20.2, C21.2, C22.2, C23.2, C24.2, C25.-, C26.-, C27.-, C28.-, FTDI231XS2.GND@16, FTDI231XS2.GND@6, IC3A.OE, IC3B.OE, IC3C.OE, IC4G$1.GND, IC5G$1.GND, IC6A.OE, IC6B.OE, IC6C.OE, J1.GND, J7_TMP3.2, MPU1.GND, S2.3, S2.4, U$2.G2, U$2.G3, U$2.VSS, U$4.G2, U$4.G3, U$4.VSS, Y2.2
- net 3.3VFTDI: now also C21.1, FTDI231XS2.!RESET, FTDI231XS2.3V3OUT, FTDI231XS2.VCCIO, R19.2, U$3.G
- net 5V: now also ATMEGA328P-AU1.AVCC, ATMEGA328P-AU1.VCC, ATMEGA328P-AU1.VCC_2, C17.1, C22.1, IC5G$1.IN, J1.VBUS, JP2.1, MPU1.VDD, R16.1, R17.1, R18.1, R20.1, U$3.D
- net A0: now also ATMEGA328P-AU1.PC0
- net A1: now also ATMEGA328P-AU1.PC1
- net A2: now also ATMEGA328P-AU1.PC2
- net A3: now also ATMEGA328P-AU1.PC3
- net A6: now also ATMEGA328P-AU1.ADC6
- net A7: now also ATMEGA328P-AU1.ADC7
- net ADO: now also MPU1.AD0
- net D2: now also ATMEGA328P-AU1.PD2
- net D3: now also ATMEGA328P-AU1.PD3
- net D4: now also ATMEGA328P-AU1.PD4
- net D5: now also ATMEGA328P-AU1.PD5
- net D6: now also ATMEGA328P-AU1.PD6
- net D7: now also ATMEGA328P-AU1.PD7
- net D8: now also ATMEGA328P-AU1.PB0
- net D9: now also ATMEGA328P-AU1.PB1
- net DTR: now also C14.1, R20.2, S2.1, S2.2
- net DTR_FTDI: now also FTDI231XS2.!DTR, R19.1, U$3.S
- net INT: now also MPU1.INT
- net MISO: now also ATMEGA328P-AU1.PB4, R14.2, R25.2, U$2.DAT0, U$4.DAT0
- net MOSI: now also ATMEGA328P-AU1.PB3, IC3B.I, IC6B.I
- net RESET: now also ATMEGA328P-AU1.PC6, R16.2
- net RX: now also FTDI231XS2.RXD, R24.1
- net RX-I: now also ATMEGA328P-AU1.PD0, R23.2
- net RXLED: now also FTDI231XS2.CBUS1
- net SCK: now also ATMEGA328P-AU1.PB5, IC3A.I, IC6A.I
- net SCL: now also ATMEGA328P-AU1.PC4, MPU1.SLC, R18.2
- net SDA: now also ATMEGA328P-AU1.PC5, C14.2, MPU1.SDA, R17.2
- net SS: now also ATMEGA328P-AU1.PB2, IC3C.I, IC6C.I
- net TX: now also FTDI231XS2.TXD, R23.1
- net TX-O: now also ATMEGA328P-AU1.PD1, R24.2
- net TXLED: now also FTDI231XS2.CBUS2
- net VCC: now also C28.+, IC3D.I, IC3D.O, IC3D.OE, IC5G$1.OUT, IC6D.I, IC6D.O, IC6D.OE, R14.1, R25.1, U$2.VDD, U$4.VDD
- net VIN: now also C27.+, D6.C, IC4G$1.IN
