File: full schematic2.sch (EAGLE design)
At the start: 61 parts, among them Q1 NPN 40V 1A SOT-23, U1 WS2812

Commit message: sd card fully laid out
Parts:
- added BUZZER1: BUZZER-PTH, SparkFun-Electromechanical:BUZZER-PTH
- added D6, D7, D8, D9: LED-IRTSAL6100, SparkFun-LED:LED-IRTSAL6100
- added IC3: 74ABT125PW, 74xx-us:74ABT125PW
- added J1, J7, J7_TMP3, J7_TMP4, J8, J8_TMP2, J8_TMP3, J9: (no value), SparkFun-Connectors:CONN_02LOCK
- added J7_NEO1, J8_NEO1: (no value), SparkFun-Connectors:CONN_03-SCREW-5MM
- added Q3: NPN 40V 1A SOT-23, semicon-smd-ipc:NPN-TRANSISTOR_SOT23
- added Q4: (no value), semicon-smd-ipc:NPN-TRANSISTOR_SOT23
- added R14: 10k, SparkFun-Resistors:0.05OHM-0603-1/5W-1%
- added R16, R17, R18, R20: 1k, SparkFun-Resistors:0.05OHM-0603-1/5W-1%
- added R19: PHOTOCELLPTH-KIT, SparkFun-Sensors:PHOTOCELLPTH-KIT
- added TMP1: (no value), SparkFun-Sensors:TMP36GT9
- added U2: WS2812, SparkFun-LED:WS2812"
Connections:
- new net BUZ-1: BUZZER1.2, J7_TMP4.2, J8_TMP3.2, Q4.C, R16.2
- new net N$10: IC3B.O, U$2.DAT1
- new net N$11: IC3C.O, U$2.CMD
- new net N$12: Q4.B, R17.1
- new net N$17: D6.C, D7.A
- new net N$24: D7.C, D8.A
- new net N$25: D8.C, D9.A
- new net N$8: U$2.G1, U$2.G4
- new net N$9: IC3A.O, U$2.CLK
- net 3.3V: now also IC3A.OE, IC3B.OE, IC3C.OE, J8_NEO1.3, Q3.E, Q4.E, U$2.G2, U$2.G3, U$2.VSS
- net 5V: now also D6.A, J7_NEO1.1, J8.1, J8_NEO1.2, J9.1, R18.1, U2.DI
- net A0: now also J1.2, J7.2, R18.2, R19.P$2
- net A1: now also TMP1.VOUT
- net BUZ+: now also BUZZER1.1, J7_TMP4.1, J8_TMP3.1, R16.1
- net D3: now also R17.2
- net D7: now also R20.2
- net D9: now also J7_NEO1.2, J8_NEO1.1, U2.VDD
- net GND: now also J1.1, J7.1, J7_NEO1.3, R19.P$1, U2.VSS
- net IR_-: now also D9.C, J8.2, J9.2, Q3.C
- net IR_LED: now also Q3.B, R20.1
- net MISO: now also R14.2, U$2.DAT0
- net MOSI: now also IC3B.I
- net SCK: now also IC3A.I
- net SS: now also IC3C.I
- net TMP+: now also J7_TMP3.1, J8_TMP2.1, TMP1.VCC
- net TMP-: now also J7_TMP3.2, J8_TMP2.2, TMP1.GND
- net VCC: now also IC3D.I, IC3D.O, IC3D.OE, R14.1, U$2.VDD
