File: 4draft_onBoard.sch (EAGLE design)
At the start: 98 parts, among them IC3 74ABT125PW, IC4 MAX4466KS, J2 USB_MINI-B_DIGIKEY, Q1 NPN 40V 1A SOT-23, U1 WS2812, U2 WS2812

Commit message: separated schematic in terms of items on board and off board so I could start to route
Parts:
- removed BUZZER, BUZZER1: BUZZER-PTH, SparkFun-Electromechanical:BUZZER-PTH
- removed D1, D2, D3, D4, D6, D7, D8, D9: LED-IRTSAL6100, SparkFun-LED:LED-IRTSAL6100
- removed IC1, IC2: (no value), linear-technology:LT1129CST5
- removed IR_LED, IR_LED1, J3_PHOTO, J3_PHOTO1, J7_BUZ, J7_BUZ1, J7_MIC, J7_MIC1, J7_TMP1, J8_TMP: (no value), SparkFun-Connectors:CONN_02LOCK
- removed J3, J7-TMP_B, J7_NEO, J7_NEO1: (no value), SparkFun-Connectors:CONN_03
- removed MK1, MK2: MIC-PTH, SparkFun-Sensors:MIC-PTH
- removed R13, R22: PHOTOCELLPTH-KIT, SparkFun-Sensors:PHOTOCELLPTH-KIT
- removed TMP36: (no value), SparkFun-Sensors:TMP36GT9
- removed U1, U2: WS2812, SparkFun-LED:WS2812"
- removed Y1: (no value), SparkFun-Clocks:RESONATORSMD-7.4X3.4
- added 3.3VREG, 5VREG: (no value), linear-technology:LT1129CST5
- added OSC: (no value), SparkFun-Clocks:RESONATORSMD-3.2X1.3
- added V_IN: (no value), SparkFun-Connectors:CONN_02LOCK
Connections:
- removed net 5V1: J7_NEO1.1, U2.DI
- removed net A4: J3_PHOTO1.2, R22.P$2
- removed net BUZ+1: BUZZER1.1, J7_BUZ1.1
- removed net BUZ-1: BUZZER1.2, J7_BUZ1.2
- removed net D1: J7_NEO1.2, U2.VDD
- removed net GND1: J3_PHOTO1.1, R22.P$1
- removed net GND2: J7_NEO1.3, U2.VSS
- removed net N$18: D1.C, D2.A
- removed net N$19: D2.C, D3.A
- removed net N$21: D3.C, D4.A
- removed net N$23: C12.+, IC1G$1.OUT, J7_5V_BACKUP.1, JP1.2
- removed net N$26: J7_MIC.1, MK1.2
- removed net N$27: J7_MIC.2, MK1.1
- removed net N$28: D6.C, D7.A
- removed net N$31: D7.C, D8.A
- removed net N$33: D8.C, D9.A
- removed net N$34: J7_MIC1.1, MK2.2
- removed net N$35: J7_MIC1.2, MK2.1
- removed net N$36: J3.2
- removed net TMP+: J8_TMP.1, TMP36.VCC
- removed net TMP-: J8_TMP.2, TMP36.GND
- new net 5REGOUT: 5VREGG$1.OUT, C12.+, J7_5V_BACKUP.1, JP1.2
- net 3.3V: now also 3.3VREGG$1.OUT, C13.+, IC3D.I, IC3D.O, IC3D.OE, R14.1, U$2.VDD; no longer ATMEGA328P-AU.GND, ATMEGA328P-AU.GND_2, ATMEGA328P-AU.GND_3, C1.2, C10.2, C11.-, C12.-, C13.-, C15.-, C2.2, C3.2, C4.2, C5.2, C6.2, C8.2, C9.2, FB2.2, FTDI231XS1.GND@16, FTDI231XS1.GND@6, IC1G$1.GND, IC2G$1.GND, IC3A.OE, IC3B.OE, IC3C.OE, J2.GND, J7-TMP_B.3, J7-TMP_B1.3, J7_TMP1.2, J8.2, J8_NEO_B.3, MPU6050.GND, Q1.E, Q2.E, S1.3, S1.4, U$2.G2, U$2.G3, U$2.VSS, Y1.2
- net 5V: now also 3.3VREGG$1.IN; no longer D1.A, D6.A, IC2G$1.IN, IR_LED.1, IR_LED1.1, J7-TMP_B.1, J7_NEO.1, U1.DI
- net A0: no longer J3_PHOTO.2, R13.P$2
- net A1: no longer TMP36.VOUT
- net BUZ+: no longer BUZZER.1, J7_BUZ.1
- net BUZ-: no longer BUZZER.2, J7_BUZ.2
- net D9: no longer J7_NEO.2, U1.VDD
- net GND: now also 3.3VREGG$1.GND, 5VREGG$1.GND, ATMEGA328P-AU.GND, ATMEGA328P-AU.GND_2, ATMEGA328P-AU.GND_3, C1.2, C10.2, C11.-, C12.-, C13.-, C15.-, C2.2, C3.2, C4.2, C5.2, C6.2, C8.2, C9.2, FB2.2, FTDI231XS1.GND@16, FTDI231XS1.GND@6, IC3A.OE, IC3B.OE, IC3C.OE, J2.GND, J7-TMP_B1.3, J8.2, J8_NEO_B.3, MPU6050.GND, OSC.2, Q1.E, Q2.E, S1.3, S1.4, U$2.G2, U$2.G3, U$2.VSS, V_IN.2; no longer J3_PHOTO.1, J7_NEO.3, R13.P$1, U1.VSS
- net IR_-: no longer D4.C, D9.C, IR_LED.2, IR_LED1.2
- net N$1: now also OSC.1; no longer Y1.1
- net N$2: now also OSC.3; no longer Y1.3
- net N$22: now also V_IN.1; no longer J7_TMP1.1
- net VCC: no longer C13.+, IC2G$1.OUT, IC3D.I, IC3D.O, IC3D.OE, R14.1, U$2.VDD
- net VIN: now also 5VREGG$1.IN; no longer IC1G$1.IN

Commit message: started board layout
Connections:
- net N$11 renamed SS_BUFF
- net N$13 renamed D-
- net N$3 renamed 2.2NF
- net N$4 renamed .UF
- net N$5 renamed 10NF
- net N$7 renamed D+
- net N$9 renamed SCK_BUFF
- removed net AREF: J8.3
- removed net N$16: C11.+, FB3.2, FTDI231XS1.VCC
- removed net N$8: U$2.G1, U$2.G4
- net GND: now also U$2.G1, U$2.G4
- net RESET: no longer J1.3, J8.13
- net RX-I: no longer J1.2
- net TX-O: no longer J1.1
- net VCC: now also C11.+, FB3.2, FTDI231XS1.VCC
- net VIN: no longer J8.15
Changed lines of the file:
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@@
 <label x="-271.78" y="124.46" size="1.778" layer="95" rot="MR0" xref="yes"/>
-</segment>
-<segment>
-<pinref part="J1" gate="G$1" pin="3"/>
-<wire x1="-200.66" y1="111.76" x2="-196.85" y2="111.76" width="0.1524" layer="91"/>
-<label x="-196.85" y="111.76" size="1.778" layer="95"/>
-</segment>
-<segment>
-<pinref part="J8" gate="G$1" pin="13"/>
-<wire x1="-170.18" y1="111.76" x2="-175.26" y2="111.76" width="0.1524" layer="91"/>
-<label x="-175.26" y="111.76" size="1.778" layer="95" rot="R180"/>
 </segment>
 </net>
@@
 <label x="-490.22" y="147.32" size="1.778" layer="95" xref="yes"/>
 </segment>
-<segment>
-<pinref part="J1" gate="G$1" pin="2"/>
-<wire x1="-200.66" y1="114.3" x2="-196.85" y2="114.3" width="0.1524" layer="91"/>
-<label x="-196.85" y="114.3" size="1.778" layer="95"/>
-</segment>
 </net>
 <net name="TX-O" class="0">
@@
 <wire x1="-501.65" y1="144.78" x2="-495.3" y2="144.78" width="0.1524" layer="91"/>
 <label x="-495.3" y="144.78" size="1.778" layer="95" xref="yes"/>
-</segment>
-<segment>
-<pinref part="J1" gate="G$1" pin="1"/>
-<wire x1="-200.66" y1="116.84" x2="-196.85" y2="116.84" width="0.1524" layer="91"/>
-<label x="-196.85" y="116.84" size="1.778" layer="95"/>
 </segment>
 </net>
@@
 </segment>
 </net>
-<net name="N$3" class="0">
+<net name="2.2NF" class="0">
 <segment>
 <pinref part="C4" gate="G$1" pin="1"/>
@@
 </segment>
 </net>
-<net name="N$4" class="0">
+<net name=".UF" class="0">
 <segment>
 <pinref part="C8" gate="G$1" pin="1"/>
@@
 </segment>
 </net>
-<net name="N$5" class="0">
+<net name="10NF" class="0">
 <segment>
 <pinref part="MPU6050" gate="G$1" pin="VLOG"/>
@@
 </segment>
 </net>
-<net name="N$7" class="0">
+<net name="D+" class="0">
 <segment>
 <pinref part="J2" gate="G$1" pin="D+"/>
@@
 </segment>
 </net>
-<net name="N$13" class="0">
+<net name="D-" class="0">
 <segment>
 <pinref part="J2" gate="G$1" pin="D-"/>
@@
 <pinref part="FTDI231XS1" gate="U$1" pin="USBDM"/>
 <wire x1="-554.99" y1="133.35" x2="-544.83" y2="137.16" width="0.1524" layer="91"/>
-</segment>
-</net>
-<net name="N$16" class="0">
-<segment>
-<wire x1="-567.69" y1="120.65" x2="-567.69" y2="140.97" width="0.1524" layer="91"/>
-<pinref part="FTDI231XS1" gate="U$1" pin="VCC"/>
-<wire x1="-567.69" y1="140.97" x2="-567.69" y2="147.32" width="0.1524" layer="91"/>
-<wire x1="-544.83" y1="147.32" x2="-567.69" y2="147.32" width="0.1524" layer="91"/>
-<pinref part="C11" gate="G$1" pin="+"/>
-<pinref part="FB3" gate="G$1" pin="2"/>
-<wire x1="-586.74" y1="140.97" x2="-567.69" y2="140.97" width="0.1524" layer="91"/>
-<junction x="-567.69" y="140.97"/>
 </segment>
 </net>
@@
 <wire x1="-464.82" y1="5.08" x2="-464.82" y2="10.16" width="0.1524" layer="91"/>
 </segment>
+<segment>
+<pinref part="U$2" gate="G1" pin="G1"/>
+<pinref part="U$2" gate="G1" pin="G4"/>
+<wire x1="-337.82" y1="236.22" x2="-320.04" y2="236.22" width="0.1524" layer="91"/>
+<wire x1="-320.04" y1="236.22" x2="-320.04" y2="235.839" width="0.1524" layer="91"/>
+</segment>
 </net>
 <net name="IR_LED" class="0">
@@
 <junction x="-491.49" y="78.74"/>
 </segment>
-<segment>
-<pinref part="J8" gate="G$1" pin="15"/>
-<wire x1="-170.18" y1="116.84" x2="-175.26" y2="116.84" width="0.1524" layer="91"/>
-<label x="-175.26" y="116.84" size="1.778" layer="95" rot="R180"/>
-</segment>
 </net>
 <net name="N$22" class="0">
@@
 <pinref part="P+3" gate="VCC" pin="VCC"/>
 </segment>
+<segment>
+<wire x1="-567.69" y1="120.65" x2="-567.69" y2="140.97" width="0.1524" layer="91"/>
+<pinref part="FTDI231XS1" gate="U$1" pin="VCC"/>
+<wire x1="-567.69" y1="140.97" x2="-567.69" y2="147.32" width="0.1524" layer="91"/>
+<wire x1="-544.83" y1="147.32" x2="-567.69" y2="147.32" width="0.1524" layer="91"/>
+<pinref part="C11" gate="G$1" pin="+"/>
+<pinref part="FB3" gate="G$1" pin="2"/>
+<wire x1="-586.74" y1="140.97" x2="-567.69" y2="140.97" width="0.1524" layer="91"/>
+<junction x="-567.69" y="140.97"/>
+</segment>
 </net>
 <net name="BUZ+" class="0">
@@
 </segment>
 </net>
-<net name="N$8" class="0">
-<segment>
-<pinref part="U$2" gate="G1" pin="G1"/>
-<pinref part="U$2" gate="G1" pin="G4"/>
-<wire x1="-337.82" y1="236.22" x2="-320.04" y2="236.22" width="0.1524" layer="91"/>
-<wire x1="-320.04" y1="236.22" x2="-320.04" y2="235.839" width="0.1524" layer="91"/>
-</segment>
-</net>
-<net name="N$9" class="0">
+<net name="SCK_BUFF" class="0">
 <segment>
 <pinref part="IC3" gate="A" pin="O"/>
@@
 </segment>
 </net>
-<net name="N$11" class="0">
+<net name="SS_BUFF" class="0">
 <segment>
 <pinref part="IC3" gate="C" pin="O"/>
@@
 </segment>
 </net>
-<net name="AREF" class="0">
-<segment>
-<pinref part="J8" gate="G$1" pin="3"/>
-<wire x1="-170.18" y1="86.36" x2="-175.26" y2="86.36" width="0.1524" layer="91"/>
-<label x="-175.26" y="86.36" size="1.778" layer="95" rot="R180"/>
-</segment>
-</net>

Commit message: shrinking board llayout
Connections:
- net GND: no longer J8.14, J8.2
Changed lines of the file:
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@@
-</segment>
-<segment>
-<pinref part="J8" gate="G$1" pin="14"/>
-<wire x1="-170.18" y1="114.3" x2="-175.26" y2="114.3" width="0.1524" layer="91"/>
-<label x="-175.26" y="114.3" size="1.778" layer="95" rot="R180"/>
 </segment>
 <segment>
@@
 </segment>
 <segment>
-<pinref part="J8" gate="G$1" pin="2"/>
-<wire x1="-170.18" y1="83.82" x2="-175.26" y2="83.82" width="0.1524" layer="91"/>
-<label x="-175.26" y="83.82" size="1.778" layer="95" rot="R180"/>
-</segment>
-<segment>

Commit message: re arranging nano layout
Connections:
- removed net N$32: C17.2, IC4.OUT, U$3.2, U$3.3
- removed net VCC: C11.+, FB1.2, FB3.2, FTDI231XS1.VCC, R19.1, R20.1
- new net AVCC: FB1.2, IC4.VCC, R19.1, R20.1
- net 5V: now also C11.+, FB3.2, FTDI231XS1.VCC
- net A6: now also C17.2, IC4.OUT, U$3.2, U$3.3; no longer IC4.VCC
Other:
- moved on the sheet: C14, C16, C17, C18, FB1, FB2, J2PHOTO_B, J5_IR_LED_B, J7-TMP_B1, J7_MIC_B, J8_BUZ_B, Q1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
