File: 5draft_onBoard_rework2.sch (EAGLE design)
At the start: 69 parts, among them IC3 74ABT125PW, IC4 MAX4466KS, J2 USB_MINI-B_DIGIKEY, Q1 NPN 40V 1A SOT-23

Commit message: redoing layout, condensing.
Connections:
- net D+_P renamed DN+_P
- net D-_N renamed DN_N
- net N$10 renamed DAT1
- net USBDM_N renamed USBD_M
- net USBDM_P renamed USBD_P
- net 5V: no longer C11.+, FB3.2, FTDI231XS1.VCC
- net SCL: now also ATMEGA328P-AU.PC5; no longer ATMEGA328P-AU.PC4
- net SDA: now also ATMEGA328P-AU.PC4; no longer ATMEGA328P-AU.PC5
- net VUSB: now also C11.+, FB3.2, FTDI231XS1.VCC
Changed lines of the file:
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@@
 <classes>
 <class number="0" name="default" width="0" drill="0">
+<clearance class="0" value="0.0508"/>
 </class>
 </classes>
@@
 <part name="R5" library="SparkFun-Resistors" deviceset="0.05OHM" device="-0603-1/5W-1%" value="27"/>
 <part name="R7" library="SparkFun-Resistors" deviceset="0.05OHM" device="-0603-1/5W-1%" value="27"/>
-<part name="SUPPLY5" library="SparkFun-PowerSymbols" deviceset="5V" device=""/>
 <part name="SUPPLY7" library="SparkFun-PowerSymbols" deviceset="5V" device=""/>
 <part name="GND21" library="SparkFun-PowerSymbols" deviceset="GND2" device=""/>
@@
 <instance part="R5" gate="G$1" x="-575.31" y="133.35"/>
 <instance part="R7" gate="G$1" x="-588.01" y="130.81"/>
-<instance part="SUPPLY5" gate="G$1" x="-604.52" y="139.7"/>
 <instance part="SUPPLY7" gate="G$1" x="-449.58" y="148.59"/>
 <instance part="GND21" gate="G$1" x="-557.53" y="105.41"/>
@@
 </segment>
 <segment>
-<wire x1="-567.69" y1="120.65" x2="-567.69" y2="140.97" width="0.1524" layer="91"/>
-<pinref part="FTDI231XS1" gate="U$1" pin="VCC"/>
-<wire x1="-567.69" y1="140.97" x2="-567.69" y2="147.32" width="0.1524" layer="91"/>
-<wire x1="-544.83" y1="147.32" x2="-567.69" y2="147.32" width="0.1524" layer="91"/>
-<pinref part="C11" gate="G$1" pin="+"/>
-<pinref part="FB3" gate="G$1" pin="2"/>
-<wire x1="-586.74" y1="140.97" x2="-567.69" y2="140.97" width="0.1524" layer="91"/>
-<junction x="-567.69" y="140.97"/>
-</segment>
-<segment>
 <pinref part="IC3" gate="D" pin="I"/>
 <wire x1="-372.11" y1="199.39" x2="-374.65" y2="199.39" width="0.1524" layer="91"/>
@@
 </segment>
 <segment>
-<pinref part="ATMEGA328P-AU" gate="A" pin="PC4"/>
-<wire x1="-285.75" y1="109.22" x2="-251.46" y2="109.22" width="0.1524" layer="91"/>
-<label x="-251.46" y="109.22" size="1.778" layer="95" xref="yes"/>
-</segment>
-<segment>
 <pinref part="J8" gate="G$1" pin="9"/>
 <wire x1="-170.18" y1="101.6" x2="-175.26" y2="101.6" width="0.1524" layer="91"/>
 <label x="-175.26" y="101.6" size="1.778" layer="95" rot="R180"/>
+</segment>
+<segment>
+<pinref part="ATMEGA328P-AU" gate="A" pin="PC5"/>
+<wire x1="-285.75" y1="106.68" x2="-264.16" y2="106.68" width="0.1524" layer="91"/>
+<label x="-264.16" y="106.68" size="1.778" layer="95" xref="yes"/>
 </segment>
 </net>
@@
 </segment>
 <segment>
-<pinref part="ATMEGA328P-AU" gate="A" pin="PC5"/>
-<wire x1="-285.75" y1="106.68" x2="-264.16" y2="106.68" width="0.1524" layer="91"/>
-<label x="-264.16" y="106.68" size="1.778" layer="95" xref="yes"/>
-</segment>
-<segment>
 <pinref part="J8" gate="G$1" pin="8"/>
 <wire x1="-170.18" y1="99.06" x2="-175.26" y2="99.06" width="0.1524" layer="91"/>
 <label x="-175.26" y="99.06" size="1.778" layer="95" rot="R180"/>
+</segment>
+<segment>
+<pinref part="ATMEGA328P-AU" gate="A" pin="PC4"/>
+<wire x1="-285.75" y1="109.22" x2="-251.46" y2="109.22" width="0.1524" layer="91"/>
+<label x="-251.46" y="109.22" size="1.778" layer="95" xref="yes"/>
 </segment>
 </net>
@@
 </segment>
 </net>
-<net name="D+_P" class="0">
+<net name="DN+_P" class="0">
 <segment>
 <pinref part="J2" gate="G$1" pin="D+"/>
@@
 </segment>
 </net>
-<net name="D-_N" class="0">
+<net name="DN_N" class="0">
 <segment>
 <pinref part="J2" gate="G$1" pin="D-"/>
@@
 </segment>
 </net>
-<net name="USBDM_P" class="0">
+<net name="USBD_P" class="0">
 <segment>
 <pinref part="R5" gate="G$1" pin="2"/>
@@
 </segment>
 </net>
-<net name="N$10" class="0">
+<net name="DAT1" class="0">
 <segment>
 <pinref part="IC3" gate="B" pin="O"/>
@@
 </segment>
 </net>
-<net name="USBDM_N" class="0">
+<net name="USBD_M" class="0">
 <segment>
 <pinref part="R7" gate="G$1" pin="2"/>
@@
 <net name="VUSB" class="0">
 <segment>
-<pinref part="SUPPLY5" gate="G$1" pin="5V"/>
-<wire x1="-604.52" y1="139.7" x2="-604.52" y2="138.43" width="0.1524" layer="91"/>
 <wire x1="-604.52" y1="138.43" x2="-604.52" y2="129.54" width="0.1524" layer="91"/>
 <wire x1="-604.52" y1="129.54" x2="-605.79" y2="128.27" width="0.1524" layer="91"/>
@@
 <wire x1="-604.52" y1="138.43" x2="-596.9" y2="138.43" width="0.1524" layer="91"/>
 <wire x1="-596.9" y1="138.43" x2="-596.9" y2="140.97" width="0.1524" layer="91"/>
-<junction x="-604.52" y="138.43"/>
-</segment>
-</net>
+</segment>
+<segment>
+<wire x1="-567.69" y1="120.65" x2="-567.69" y2="140.97" width="0.1524" layer="91"/>
+<pinref part="FTDI231XS1" gate="U$1" pin="VCC"/>
+<wire x1="-567.69" y1="140.97" x2="-567.69" y2="147.32" width="0.1524" layer="91"/>
+<wire x1="-544.83" y1="147.32" x2="-567.69" y2="147.32" width="0.1524" layer="91"/>
+<pinref part="C11" gate="G$1" pin="+"/>
+<pinref part="FB3" gate="G$1" pin="2"/>
+<wire x1="-586.74" y1="140.97" x2="-567.69" y2="140.97" width="0.1524" layer="91"/>
+<junction x="-567.69" y="140.97"/>
+</segment>
+</net>

Commit message: 3rd draft, close to final. FTDI might need to be reworked. and there is a bug. I do not know why AVCC is routed to VCC when it should not be, cannot find net causing issue
Connections:
- net N$17 renamed MICNET1K
- net N$24 renamed MIC_IN_C14
- net N$25 renamed MIC_IN+
- net D6: now also J9_PIR1.1
- net D7: no longer J9_PIR1.1
- net GND: now also J2.SHIELD
